File: cheaponder.kicad_pcb (KiCad board)
At the start: 2 copper layers, 18 x 22.5 mm, 32 parts, among them J1 B+, J2 B-, Q1 FS8205A, U1 TP4057, U2 DW01A, U3 TPS63900, U4 ESP32-S3-Zero Devboard

Commit message: Implement some of Max' Feedback
Routing:
- net GND: track 21.9 -> 19.8 mm, vias 16 -> 22
Other:
- board text added: "v0.2"
- board text removed: "v0.1"
Changed lines of the file:
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@@
 		)
 	)
-	(gr_text "v0.1"
+	(gr_text "v0.2"
 		(at 72.7 125.2 0)
 		(layer "F.SilkS")
@@
 	)
 	(segment
+		(start 87.387501 111.3)
+		(end 86.671625 111.922418)
+		(width 0.25)
+		(layer "F.Cu")
+		(net 2)
+	)
+	(segment
+		(start 76.059374 104.559374)
+		(end 75.6 104.9)
+		(width 1)
+		(layer "F.Cu")
+		(net 2)
+	)
+	(segment
+		(start 80.2 118.133551)
+		(end 80.751938 118.081233)
+		(width 0.25)
+		(layer "F.Cu")
+		(net 2)
+	)
+	(segment
+		(start 75.6 104.9)
+		(end 75.336965 105.436965)
+		(width 1)
+		(layer "F.Cu")
+		(net 2)
+	)
+	(segment
+		(start 79.055444 118.8)
+		(end 79.246224 118.546224)
+		(width 0.25)
+		(layer "F.Cu")
+		(net 2)
+	)
+	(segment
 		(start 82.203174 108.257151)
 		(end 81.2125 108.2575)
@@
 	)
 	(segment
-		(start 87.387501 111.3)
-		(end 86.671625 111.922418)
-		(width 0.25)
-		(layer "F.Cu")
-		(net 2)
-	)
-	(segment
-		(start 76.059374 104.559374)
-		(end 75.6 104.9)
-		(width 1)
-		(layer "F.Cu")
-		(net 2)
-	)
-	(segment
-		(start 80.2 118.133551)
-		(end 80.751938 118.081233)
-		(width 0.25)
-		(layer "F.Cu")
-		(net 2)
-	)
-	(segment
-		(start 75.6 104.9)
-		(end 75.336965 105.436965)
-		(width 1)
-		(layer "F.Cu")
-		(net 2)
-	)
-	(segment
-		(start 79.055444 118.8)
-		(end 79.246224 118.546224)
-		(width 0.25)
-		(layer "F.Cu")
-		(net 2)
-	)
-	(segment
 		(start 78.225 121)
 		(end 78.8 119.3375)
@@
 	)
 	(segment
-		(start 85.013262 107.927565)
-		(end 82.203174 108.257151)
-		(width 0.25)
-		(layer "F.Cu")
-		(net 2)
-	)
-	(segment
 		(start 79.7 118.272554)
 		(end 79.9 118.192524)
@@
 	)
 	(segment
+		(start 82.9 108.175423)
+		(end 82.203174 108.257151)
+		(width 0.25)
+		(layer "F.Cu")
+		(net 2)
+	)
+	(segment
 		(start 85.875 113.0375)
 		(end 86.2 113.0375)
@@
 	)
 	(via
+		(at 83.956367 108.047029)
+		(size 0.6)
+		(drill 0.3)
+		(layers "F.Cu" "B.Cu")
+		(free yes)
+		(net 2)
+	)
+	(via
+		(at 80 109.4)
+		(size 0.6)
+		(drill 0.3)
+		(layers "F.Cu" "B.Cu")
+		(free yes)
+		(net 2)
+	)
+	(via
 		(at 86.2 114.2)
 		(size 0.6)
@@
 	)
 	(via
+		(at 80 107.1)
+		(size 0.6)
+		(drill 0.3)
+		(layers "F.Cu" "B.Cu")
+		(free yes)
+		(net 2)
+	)
+	(via
 		(at 85.8 115.8)
 		(size 0.6)
@@
 	)
 	(via
+		(at 80.3 115)
+		(size 0.6)
+		(drill 0.3)
+		(layers "F.Cu" "B.Cu")
+		(free yes)
+		(net 2)
+	)
+	(via
 		(at 83.9 113.4)
 		(size 0.6)
@@
 	)
 	(via
+		(at 78.1 109.5)
+		(size 0.6)
+		(drill 0.3)
+		(layers "F.Cu" "B.Cu")
+		(free yes)
+		(net 2)
+	)
+	(via
 		(at 77.3 113)
 		(size 0.6)
@@
 		(size 0.6)
 		(drill 0.3)
+		(layers "F.Cu" "B.Cu")
+		(free yes)
+		(net 2)
+	)
+	(via
+		(at 82.9 108.175423)
+		(size 0.6)
+		(drill 0.3)
