File: cheaponder.kicad_sch (KiCad schematic)
At the start: 32 parts, among them J1 B+, J2 B-, Q1 FS8205A, U1 TP4057, U2 DW01A, U3 TPS63900, U4 ESP32-S3-Zero Devboard

Commit message: Update to KiCAD 9
Changed lines of the file:
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@@
 (kicad_sch
-	(version 20231120)
+	(version 20250114)
 	(generator "eeschema")
-	(generator_version "8.0")
+	(generator_version "9.0")
 	(paper "A4")
+	(rectangle
+		(start 50.8 101.6)
+		(end 114.3 165.1)
+		(stroke
+			(width 0)
+			(type dash_dot)
+		)
+		(fill
+			(type none)
+		)
+	)
+	(rectangle
+		(start 127 38.1)
+		(end 203.2 88.9)
+		(stroke
+			(width 0)
+			(type dash_dot)
+		)
+		(fill
+			(type none)
+		)
+	)
+	(rectangle
+		(start 127 101.6)
+		(end 241.3 152.4)
+		(stroke
+			(width 0)
+			(type dash_dot)
+		)
+		(fill
+			(type none)
+		)
+	)
+	(rectangle
+		(start 50.8 38.1)
+		(end 114.3 88.9)
+		(stroke
+			(width 0)
+			(type dash_dot)
+		)
+		(fill
+			(type none)
+		)
+	)
+	(text "Charging"
+		(exclude_from_sim no)
+		(at 113.538 86.36 0)
+		(effects
+			(font
+				(size 1.27 1.27)
+			)
+			(justify right top)
+		)
+	)
+	(text "ESR target: ~1mOhm total"
+		(exclude_from_sim no)
+		(at 161.29 124.714 0)
+		(effects
+			(font
+				(size 1.27 1.27)
+				(color 194 0 194 1)
+			)
+		)
+	)
+	(text "1k6 = 500mA"
+		(exclude_from_sim no)
+		(at 94.488 79.502 0)
+		(effects
+			(font
+				(size 1.27 1.27)
+			)
+		)
+	)
+	(text "Power Supply"
+		(exclude_from_sim no)
+		(at 240.538 149.86 0)
+		(effects
+			(font
+				(size 1.27 1.27)
+			)
+			(justify right top)
+		)
+	)
+	(text "Wi-Fi Module"
+		(exclude_from_sim no)
+		(at 113.538 162.814 0)
+		(effects
+			(font
+				(size 1.27 1.27)
+			)
+			(justify right top)
+		)
+	)
+	(text "Bat Protection"
+		(exclude_from_sim no)
+		(at 202.184 86.614 0)
+		(effects
+			(font
+				(size 1.27 1.27)
+			)
+			(justify right top)
+		)
+	)
+	(text "ESR target: ~3.7mOhm total"
+		(exclude_from_sim no)
+		(at 210.82 124.714 0)
+		(effects
+			(font
+				(size 1.27 1.27)
+				(color 194 0 194 1)
+			)
+		)
+	)
+	(text "https://webench.ti.com/appinfo/webench/scripts/SDP.cgi?ID=ED25D392B281E2A0"
+		(exclude_from_sim no)
+		(at 173.736 107.442 0)
+		(effects
+			(font
+				(size 1.27 1.27)
+			)
+		)
+	)
 	(junction
 		(at 182.88 57.15)
@@
 		(at 71.12 132.08)
 	)
-	(bus_entry
-		(at 88.9 44.45)
-		(size 2.54 2.54)
-		(stroke
-			(width 0)
-			(type default)
-		)
-	)
 	(wire
 		(pts
@@
 		)
 	)
-	(rectangle
-		(start 50.8 101.6)
-		(end 114.3 165.1)
-		(stroke
-			(width 0)
-			(type dash_dot)
-		)
-		(fill
-			(type none)
-		)
-	)
-	(rectangle
-		(start 127 38.1)
-		(end 203.2 88.9)
-		(stroke
-			(width 0)
-			(type dash_dot)
-		)
-		(fill
-			(type none)
-		)
-	)
-	(rectangle
-		(start 127 101.6)
-		(end 241.3 152.4)
-		(stroke
-			(width 0)
-			(type dash_dot)
-		)
-		(fill
-			(type none)
-		)
-	)
-	(rectangle
-		(start 50.8 38.1)
-		(end 114.3 88.9)
-		(stroke
-			(width 0)
-			(type dash_dot)
-		)
-		(fill
-			(type none)
-		)
-	)
-	(text "Charging"
-		(exclude_from_sim no)
-		(at 113.538 86.36 0)
-		(effects
-			(font
-				(size 1.27 1.27)
-			)
-			(justify right top)
-		)
-	)
-	(text "ESR target: ~1mOhm total"
-		(exclude_from_sim no)
-		(at 161.29 124.714 0)
-		(effects
-			(font
-				(size 1.27 1.27)
-				(color 194 0 194 1)
-			)
-		)
-	)
-	(text "1k6 = 500mA"
-		(exclude_from_sim no)
-		(at 94.488 79.502 0)
-		(effects
-			(font
-				(size 1.27 1.27)
-			)
-		)
-	)
-	(text "Power Supply"
-		(exclude_from_sim no)
-		(at 240.538 149.86 0)
-		(effects
-			(font
-				(size 1.27 1.27)
-			)
-			(justify right top)
-		)
-	)
-	(text "Wi-Fi Module"
-		(exclude_from_sim no)
-		(at 113.538 162.814 0)
-		(effects
-			(font
-				(size 1.27 1.27)
-			)
-			(justify right top)
-		)
-	)
-	(text "Bat Protection"
-		(exclude_from_sim no)
-		(at 202.184 86.614 0)
-		(effects
-			(font
-				(size 1.27 1.27)
-			)
-			(justify right top)
-		)
-	)
-	(text "ESR target: ~3.7mOhm total"
-		(exclude_from_sim no)
-		(at 210.82 124.714 0)
-		(effects
-			(font
-				(size 1.27 1.27)
-				(color 194 0 194 1)
-			)
-		)
-	)
-	(text "https://webench.ti.com/appinfo/webench/scripts/SDP.cgi?ID=ED25D392B281E2A0"
-		(exclude_from_sim no)
-		(at 173.736 107.442 0)
-		(effects
-			(font
-				(size 1.27 1.27)
-			)
-		)
-	)
 	(label "DW_CS"
 		(at 182.88 77.47 0)
-		(fields_autoplaced yes)
 		(effects
 			(font
@@
 	(label "L2"
 		(at 177.8 135.89 0)
-		(fields_autoplaced yes)
 		(effects
 			(font
@@
 	(label "ESP_LED"
 		(at 91.44 139.7 0)
-		(fields_autoplaced yes)
 		(effects
 			(font
@@
 	(label "DW_OC"
 		(at 176.53 69.85 180)
-		(fields_autoplaced yes)
 		(effects
 			(font
@@
 	(label "+VIN"
 		(at 147.32 118.11 90)
-		(fields_autoplaced yes)
 		(effects
 			(font
@@
 	(label "DW_OD"
 		(at 176.53 64.77 180)
-		(fields_autoplaced yes)
 		(effects
 			(font
@@
 	(label "TP_STBY"
 		(at 73.66 69.85 180)
-		(fields_autoplaced yes)
 		(effects
 			(font
@@
 	(label "VBAT_MON"
 		(at 71.12 124.46 180)
-		(fields_autoplaced yes)
 		(effects
 			(font
@@
 	(label "TP_CHRG"
 		(at 73.66 64.77 180)
-		(fields_autoplaced yes)
 		(effects
 			(font
@@
 	(label "L1"
 		(at 177.8 130.81 0)
-		(fields_autoplaced yes)
 		(effects
 			(font
@@
 		)
 	)
+	(embedded_fonts no)
 )

Commit message: Fix link and add comment
Other:
- note added: "De-Solder LDO from ESP32!"
- note added: "https://webench.ti.com/appinfo/webench/scripts/SDP.cgi?ID=E00DE86EFB21CDE4"
- note removed: "https://webench.ti.com/appinfo/webench/scripts/SDP.cgi?ID=ED25D392B281E2A0"
Changed lines of the file:
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@@
+		)
+	)
+	(text "De-Solder LDO from ESP32!"
+		(exclude_from_sim no)
+		(at 98.806 117.348 0)
+		(effects
+			(font
+				(size 1.27 1.27)
+				(thickness 0.254)
+				(bold yes)
+				(color 255 0 0 1)
+			)
 		)
 	)
@@
 		)
 	)
-	(text "https://webench.ti.com/appinfo/webench/scripts/SDP.cgi?ID=ED25D392B281E2A0"
+	(text "https://webench.ti.com/appinfo/webench/scripts/SDP.cgi?ID=E00DE86EFB21CDE4"
 		(exclude_from_sim no)
 		(at 173.736 107.442 0)

Commit message: Relayout to accomodate bigger cap and put LEDs where we can see them
Parts:
- C3: footprint Capacitor_SMD:C_0603_1608Metric -> Capacitor_SMD:C_0805_2012Metric
Changed lines of the file:
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@@
 			)
 		)
-		(property "Footprint" "Capacitor_SMD:C_0603_1608Metric"
+		(property "Footprint" "Capacitor_SMD:C_0805_2012Metric"
 			(at 101.9048 71.12 0)
 			(effects
